File: kicad/binaryclock.sch (KiCad schematic (older format))
At the start: 7 parts, among them IC1 ATMEGA328P-PU, SW1 Reset, Y1 16MHz

Commit message: update kicad
Parts:
- added U? (x3): 74HC595, symbol 74HC595
Connections:
- net at IC1.12 ((PCINT22/OC0A/AIN0)PD6): now also U?.11 (SRCLK), U?.11 (SRCLK), U?.11 (SRCLK)
- net at IC1.13 ((PCINT23/AIN1)PD7): now also U?.14 (SER)
- net at IC1.14 ((PCINT0/CLKO/ICP1)PB0): now also U?.12 (RCLK), U?.12 (RCLK), U?.12 (RCLK)
- new net: U?.14 (SER), U?.9 (~QH) (x2)
- new net GND: U?.8 (GND), U?.8 (GND), U?.8 (GND)
- new net VCC: U?.16 (VCC), U?.16 (VCC), U?.16 (VCC)
Changed lines of the file:
@@
+	1    0    0    -1
+$EndComp
+$Comp
+L Earth #PWR?
+U 1 1 58ED2D1B
+P 2050 4500
+F 0 "#PWR?" H 2050 4250 50  0001 C CNN
+F 1 "Earth" H 2050 4350 50  0001 C CNN
+F 2 "" H 2050 4500 50  0001 C CNN
+F 3 "" H 2050 4500 50  0001 C CNN
+	1    2050 4500
+	1    0    0    -1
+$EndComp
+$Comp
+L Earth #PWR?
+U 1 1 58ED2D67
+P 6000 3650
+F 0 "#PWR?" H 6000 3400 50  0001 C CNN
+F 1 "Earth" H 6000 3500 50  0001 C CNN
+F 2 "" H 6000 3650 50  0001 C CNN
+F 3 "" H 6000 3650 50  0001 C CNN
+	1    6000 3650
+	1    0    0    -1
+$EndComp
+$Comp
+L 74HC595 U?
+U 1 1 58EE5DCD
+P 2100 6450
+F 0 "U?" H 2250 7050 50  0000 C CNN
+F 1 "74HC595" H 2100 5850 50  0000 C CNN
+F 2 "" H 2100 6450 50  0001 C CNN
+F 3 "" H 2100 6450 50  0001 C CNN
+	1    2100 6450
+	1    0    0    -1
+$EndComp
+$Comp
+L 74HC595 U?
+U 1 1 58EE5E60
+P 2100 7850
+F 0 "U?" H 2250 8450 50  0000 C CNN
+F 1 "74HC595" H 2100 7250 50  0000 C CNN
+F 2 "" H 2100 7850 50  0001 C CNN
+F 3 "" H 2100 7850 50  0001 C CNN
+	1    2100 7850
+	1    0    0    -1
+$EndComp
+$Comp
+L 74HC595 U?
+U 1 1 58EE5F30
+P 2100 9250
+F 0 "U?" H 2250 9850 50  0000 C CNN
+F 1 "74HC595" H 2100 8650 50  0000 C CNN
+F 2 "" H 2100 9250 50  0001 C CNN
+F 3 "" H 2100 9250 50  0001 C CNN
+	1    2100 9250
 	1    0    0    -1
 $EndComp
@@
 	4700 1450 4700 4650
 Connection ~ 4700 3300
-$Comp
-L Earth #PWR?
-U 1 1 58ED2D1B
-P 2050 4500
-F 0 "#PWR?" H 2050 4250 50  0001 C CNN
-F 1 "Earth" H 2050 4350 50  0001 C CNN
-F 2 "" H 2050 4500 50  0001 C CNN
-F 3 "" H 2050 4500 50  0001 C CNN
-	1    2050 4500
-	1    0    0    -1
-$EndComp
-$Comp
-L Earth #PWR?
-U 1 1 58ED2D67
-P 6000 3650
-F 0 "#PWR?" H 6000 3400 50  0001 C CNN
-F 1 "Earth" H 6000 3500 50  0001 C CNN
-F 2 "" H 6000 3650 50  0001 C CNN
-F 3 "" H 6000 3650 50  0001 C CNN
-	1    6000 3650
-	1    0    0    -1
-$EndComp
+Wire Wire Line
+	5450 5500 800  5500
+Wire Wire Line
+	800  5500 800  9000
+Wire Wire Line
+	800  6200 1400 6200
+Wire Wire Line
+	800  7600 1400 7600
+Connection ~ 800  6200
+Wire Wire Line
+	800  9000 1400 9000
+Connection ~ 800  7600
+Wire Wire Line
+	4200 4050 5450 4050
+Wire Wire Line
+	5450 4050 5450 5500
+Wire Wire Line
+	4200 4150 5550 4150
+Wire Wire Line
+	5550 4150 5550 5600
+Wire Wire Line
+	5550 5600 1400 5600
+Wire Wire Line
+	1400 5600 1400 6000
+Wire Wire Line
+	2800 6900 2800 7150
+Wire Wire Line
+	2800 7150 1400 7150
+Wire Wire Line
+	1400 7150 1400 7400
+Wire Wire Line
+	2800 8300 2800 8550
+Wire Wire Line
+	2800 8550 1400 8550
+Wire Wire Line
+	1400 8550 1400 8800
+Wire Wire Line
+	4200 1850 6200 1850
+Wire Wire Line
+	6200 1850 6200 5700
+Wire Wire Line
+	6200 5700 900  5700
+Wire Wire Line
+	900  5700 900  9300
+Wire Wire Line
+	900  6500 1400 6500
+Wire Wire Line
+	900  7900 1400 7900
+Connection ~ 900  6500
+Wire Wire Line
+	900  9300 1400 9300
+Connection ~ 900  7900
 $EndSCHEMATC

Commit message: update kicad
Parts:
- added D? (x24): LED, symbol LED
- added RN? (x3): R_Network08, Resistors_THT:R_Array_SIP9, symbol R_Network08
Connections:
- net Earth: now also RN?.1 (common), RN?.1 (common), RN?.1 (common)
- net at U?.1 (QB): now also D?.2 (A) (x3)
- net at U?.15 (QA): now also D?.2 (A) (x3)
- net at U?.2 (QC): now also D?.2 (A) (x3)
- net at U?.3 (QD): now also D?.2 (A) (x3)
- net at U?.4 (QE): now also D?.2 (A) (x3)
- net at U?.5 (QF): now also D?.2 (A) (x3)
- net at U?.6 (QG): now also D?.2 (A) (x3)
- net at U?.7 (QH): now also D?.2 (A) (x3)
- new net: D?.1 (K), RN?.2 (R1) (x3)
- new net: D?.1 (K), RN?.3 (R2) (x3)
- new net: D?.1 (K), RN?.4 (R3) (x3)
- new net: D?.1 (K), RN?.5 (R4) (x3)
- new net: D?.1 (K), RN?.6 (R5) (x3)
- new net: D?.1 (K), RN?.7 (R6) (x3)
- new net: D?.1 (K), RN?.8 (R7) (x3)
- new net: D?.1 (K), RN?.9 (R8) (x3)

Commit message: update kicad
Parts:
- gave numbers to parts that had none: 30
Changed lines of the file:
@@
 encoding utf-8
 Sheet 1 1
-Title "Simon"
-Date "2016-03-25"
+Title "Binaryclock"
+Date "2017-04-13"
 Rev "0.2"
 Comp ""
@@
 $EndComp
 $Comp
-L +5V #PWR1
+L +5V #PWR01
 U 1 1 5683D91E
 P 2050 1350
-F 0 "#PWR1" H 2050 1200 50  0001 C CNN
+F 0 "#PWR01" H 2050 1200 50  0001 C CNN
 F 1 "+5V" H 2050 1490 50  0000 C CNN
 F 2 "" H 2050 1350 50  0000 C CNN
@@
 $EndComp
 $Comp
-L Earth #PWR?
+L Earth #PWR02
 U 1 1 58ED2D1B
 P 2050 4500
-F 0 "#PWR?" H 2050 4250 50  0001 C CNN
+F 0 "#PWR02" H 2050 4250 50  0001 C CNN
 F 1 "Earth" H 2050 4350 50  0001 C CNN
 F 2 "" H 2050 4500 50  0001 C CNN
@@
 $EndComp
 $Comp
-L Earth #PWR?
+L Earth #PWR03
 U 1 1 58ED2D67
 P 6000 3650
-F 0 "#PWR?" H 6000 3400 50  0001 C CNN
+F 0 "#PWR03" H 6000 3400 50  0001 C CNN
 F 1 "Earth" H 6000 3500 50  0001 C CNN
 F 2 "" H 6000 3650 50  0001 C CNN
@@
 $EndComp
 $Comp
-L 74HC595 U?
+L 74HC595 U1
 U 1 1 58EE5DCD
 P 2100 6450
-F 0 "U?" H 2250 7050 50  0000 C CNN
+F 0 "U1" H 2250 7050 50  0000 C CNN
 F 1 "74HC595" H 2100 5850 50  0000 C CNN
 F 2 "" H 2100 6450 50  0001 C CNN
@@
 $EndComp
 $Comp
-L 74HC595 U?
+L 74HC595 U2
 U 1 1 58EE5E60
 P 2100 7850
-F 0 "U?" H 2250 8450 50  0000 C CNN
+F 0 "U2" H 2250 8450 50  0000 C CNN
 F 1 "74HC595" H 2100 7250 50  0000 C CNN
 F 2 "" H 2100 7850 50  0001 C CNN
@@
 $EndComp
 $Comp
-L 74HC595 U?
+L 74HC595 U3
 U 1 1 58EE5F30
 P 2100 9250
-F 0 "U?" H 2250 9850 50  0000 C CNN
+F 0 "U3" H 2250 9850 50  0000 C CNN
 F 1 "74HC595" H 2100 8650 50  0000 C CNN
 F 2 "" H 2100 9250 50  0001 C CNN
@@
 $EndComp
 $Comp
-L R_Network08 RN?
+L R_Network08 RN1
 U 1 1 58EF59E2
 P 3900 6400
-F 0 "RN?" V 3400 6400 50  0000 C CNN
+F 0 "RN1" V 3400 6400 50  0000 C CNN
 F 1 "R_Network08" V 4300 6400 50  0000 C CNN
 F 2 "Resistors_THT:R_Array_SIP9" V 4375 6400 50  0001 C CNN
@@
 $EndComp
 $Comp
-L R_Network08 RN?
+L R_Network08 RN2
 U 1 1 58EF5AD8
 P 3900 7800
-F 0 "RN?" V 3400 7800 50  0000 C CNN
+F 0 "RN2" V 3400 7800 50  0000 C CNN
 F 1 "R_Network08" V 4300 7800 50  0000 C CNN
 F 2 "Resistors_THT:R_Array_SIP9" V 4375 7800 50  0001 C CNN
@@
 $EndComp
 $Comp
-L R_Network08 RN?
+L R_Network08 RN3
 U 1 1 58EF5B60
 P 3900 9200
-F 0 "RN?" V 3400 9200 50  0000 C CNN
+F 0 "RN3" V 3400 9200 50  0000 C CNN
 F 1 "R_Network08" V 4300 9200 50  0000 C CNN
 F 2 "Resistors_THT:R_Array_SIP9" V 4375 9200 50  0001 C CNN
@@
 Connection ~ 4300 7400
 $Comp
-L Earth #PWR?
+L Earth #PWR04
 U 1 1 58EF5DC6
 P 4550 8800
-F 0 "#PWR?" H 4550 8550 50  0001 C CNN
+F 0 "#PWR04" H 4550 8550 50  0001 C CNN
 F 1 "Earth" H 4550 8650 50  0001 C CNN
 F 2 "" H 4550 8800 50  0001 C CNN
@@
 Connection ~ 4300 8800
 $Comp
-L LED D?
+L LED D1
 U 1 1 58EF5FCE
 P 3250 6000
-F 0 "D?" H 3250 6100 50  0000 C CNN
+F 0 "D1" H 3250 6100 50  0000 C CNN
 F 1 "LED" H 3250 5900 50  0000 C CNN
 F 2 "" H 3250 6000 50  0001 C CNN
@@
 $EndComp
 $Comp
-L LED D?
+L LED D2
 U 1 1 58EF6047
 P 3250 6100
-F 0 "D?" H 3250 6200 50  0000 C CNN
+F 0 "D2" H 3250 6200 50  0000 C CNN
 F 1 "LED" H 3250 6000 50  0000 C CNN
 F 2 "" H 3250 6100 50  0001 C CNN
@@
 $EndComp
 $Comp
-L LED D?
+L LED D3
 U 1 1 58EF6093
 P 3250 6200
-F 0 "D?" H 3250 6300 50  0000 C CNN
+F 0 "D3" H 3250 6300 50  0000 C CNN
 F 1 "LED" H 3250 6100 50  0000 C CNN
 F 2 "" H 3250 6200 50  0001 C CNN
@@
 $EndComp
 $Comp
-L LED D?
+L LED D4
 U 1 1 58EF60D3
 P 3250 6300
-F 0 "D?" H 3250 6400 50  0000 C CNN
+F 0 "D4" H 3250 6400 50  0000 C CNN
 F 1 "LED" H 3250 6200 50  0000 C CNN
 F 2 "" H 3250 6300 50  0001 C CNN
@@
 $EndComp
 $Comp
-L LED D?
+L LED D5
 U 1 1 58EF6148
 P 3250 6400
-F 0 "D?" H 3250 6500 50  0000 C CNN
+F 0 "D5" H 3250 6500 50  0000 C CNN
 F 1 "LED" H 3250 6300 50  0000 C CNN
 F 2 "" H 3250 6400 50  0001 C CNN
@@
 $EndComp
 $Comp
-L LED D?
+L LED D6
 U 1 1 58EF6192
 P 3250 6500
-F 0 "D?" H 3250 6600 50  0000 C CNN
+F 0 "D6" H 3250 6600 50  0000 C CNN
 F 1 "LED" H 3250 6400 50  0000 C CNN
 F 2 "" H 3250 6500 50  0001 C CNN
@@
 $EndComp
 $Comp
-L LED D?
+L LED D7
 U 1 1 58EF61DB
 P 3250 6600
-F 0 "D?" H 3250 6700 50  0000 C CNN
+F 0 "D7" H 3250 6700 50  0000 C CNN
 F 1 "LED" H 3250 6500 50  0000 C CNN
 F 2 "" H 3250 6600 50  0001 C CNN
@@
 $EndComp
 $Comp
-L LED D?
+L LED D8
 U 1 1 58EF6227
 P 3250 6700
-F 0 "D?" H 3250 6800 50  0000 C CNN
+F 0 "D8" H 3250 6800 50  0000 C CNN
 F 1 "LED" H 3250 6600 50  0000 C CNN
 F 2 "" H 3250 6700 50  0001 C CNN
@@
 $EndComp
 $Comp
-L LED D?
+L LED D9
 U 1 1 58EF62EA
 P 3250 7400
-F 0 "D?" H 3250 7500 50  0000 C CNN
+F 0 "D9" H 3250 7500 50  0000 C CNN
 F 1 "LED" H 3250 7300 50  0000 C CNN
 F 2 "" H 3250 7400 50  0001 C CNN
@@
 $EndComp
 $Comp
-L LED D?
+L LED D10
 U 1 1 58EF635E
 P 3250 7500
-F 0 "D?" H 3250 7600 50  0000 C CNN
+F 0 "D10" H 3250 7600 50  0000 C CNN
 F 1 "LED" H 3250 7400 50  0000 C CNN
 F 2 "" H 3250 7500 50  0001 C CNN
@@
 $EndComp
 $Comp
-L LED D?
+L LED D11
 U 1 1 58EF63B3
 P 3250 7600
-F 0 "D?" H 3250 7700 50  0000 C CNN
+F 0 "D11" H 3250 7700 50  0000 C CNN
 F 1 "LED" H 3250 7500 50  0000 C CNN
 F 2 "" H 3250 7600 50  0001 C CNN
@@
 $EndComp
 $Comp
-L LED D?
+L LED D12
 U 1 1 58EF640B
 P 3250 7700
-F 0 "D?" H 3250 7800 50  0000 C CNN
+F 0 "D12" H 3250 7800 50  0000 C CNN
 F 1 "LED" H 3250 7600 50  0000 C CNN
 F 2 "" H 3250 7700 50  0001 C CNN
@@
 $EndComp
 $Comp
-L LED D?
+L LED D13
 U 1 1 58EF6466
 P 3250 7800
-F 0 "D?" H 3250 7900 50  0000 C CNN
+F 0 "D13" H 3250 7900 50  0000 C CNN
 F 1 "LED" H 3250 7700 50  0000 C CNN
 F 2 "" H 3250 7800 50  0001 C CNN
@@
 $EndComp
 $Comp
-L LED D?
+L LED D14
 U 1 1 58EF64C4
 P 3250 7900
-F 0 "D?" H 3250 8000 50  0000 C CNN
+F 0 "D14" H 3250 8000 50  0000 C CNN
 F 1 "LED" H 3250 7800 50  0000 C CNN
 F 2 "" H 3250 7900 50  0001 C CNN
@@
 $EndComp
 $Comp
-L LED D?
+L LED D15
 U 1 1 58EF6525
 P 3250 8000
-F 0 "D?" H 3250 8100 50  0000 C CNN
+F 0 "D15" H 3250 8100 50  0000 C CNN
 F 1 "LED" H 3250 7900 50  0000 C CNN
 F 2 "" H 3250 8000 50  0001 C CNN
@@
 $EndComp
 $Comp
-L LED D?
+L LED D16
 U 1 1 58EF6589
 P 3250 8100
-F 0 "D?" H 3250 8200 50  0000 C CNN
+F 0 "D16" H 3250 8200 50  0000 C CNN
 F 1 "LED" H 3250 8000 50  0000 C CNN
 F 2 "" H 3250 8100 50  0001 C CNN
@@
 $EndComp
 $Comp
-L LED D?
+L LED D17
 U 1 1 58EF65F0
 P 3250 8800
-F 0 "D?" H 3250 8900 50  0000 C CNN
+F 0 "D17" H 3250 8900 50  0000 C CNN
 F 1 "LED" H 3250 8700 50  0000 C CNN
 F 2 "" H 3250 8800 50  0001 C CNN
@@
 $EndComp
 $Comp
-L LED D?
+L LED D18
 U 1 1 58EF6672
 P 3250 8900
-F 0 "D?" H 3250 9000 50  0000 C CNN
+F 0 "D18" H 3250 9000 50  0000 C CNN
 F 1 "LED" H 3250 8800 50  0000 C CNN
 F 2 "" H 3250 8900 50  0001 C CNN
@@
 $EndComp
 $Comp
-L LED D?
+L LED D19
 U 1 1 58EF66DF
 P 3250 9000
-F 0 "D?" H 3250 9100 50  0000 C CNN
+F 0 "D19" H 3250 9100 50  0000 C CNN
 F 1 "LED" H 3250 8900 50  0000 C CNN
 F 2 "" H 3250 9000 50  0001 C CNN
@@
 $EndComp
 $Comp
-L LED D?
+L LED D20
 U 1 1 58EF674F
 P 3250 9100
-F 0 "D?" H 3250 9200 50  0000 C CNN
+F 0 "D20" H 3250 9200 50  0000 C CNN
 F 1 "LED" H 3250 9000 50  0000 C CNN
 F 2 "" H 3250 9100 50  0001 C CNN
@@
 $EndComp
 $Comp
-L LED D?
+L LED D21
 U 1 1 58EF67C2
 P 3250 9200
-F 0 "D?" H 3250 9300 50  0000 C CNN
+F 0 "D21" H 3250 9300 50  0000 C CNN
 F 1 "LED" H 3250 9100 50  0000 C CNN
 F 2 "" H 3250 9200 50  0001 C CNN
@@
 $EndComp
 $Comp
-L LED D?
+L LED D22
 U 1 1 58EF69B6
 P 3250 9300
-F 0 "D?" H 3250 9400 50  0000 C CNN
+F 0 "D22" H 3250 9400 50  0000 C CNN
 F 1 "LED" H 3250 9200 50  0000 C CNN
 F 2 "" H 3250 9300 50  0001 C CNN
@@
 $EndComp
 $Comp
-L LED D?
+L LED D23
 U 1 1 58EF6A2F
 P 3250 9400
-F 0 "D?" H 3250 9500 50  0000 C CNN
+F 0 "D23" H 3250 9500 50  0000 C CNN
 F 1 "LED" H 3250 9300 50  0000 C CNN
 F 2 "" H 3250 9400 50  0001 C CNN
@@
 $EndComp
 $Comp
-L LED D?
+L LED D24
 U 1 1 58EF6AAB
 P 3250 9500
-F 0 "D?" H 3250 9600 50  0000 C CNN
+F 0 "D24" H 3250 9600 50  0000 C CNN
 F 1 "LED" H 3250 9400 50  0000 C CNN
 F 2 "" H 3250 9500 50  0001 C CNN

Commit message: update kicad
Connections:
- net +5V: now also U1.10 (SRCLR), U2.10 (SRCLR), U3.10 (SRCLR)
- net Earth: now also U1.13 (G), U2.13 (G), U3.13 (G)
Other:
- moved on the sheet: C1, C2, C3, IC1, R1, SW1, Y1

Commit message: update kicad
Parts:
- added U?: PCF8563, symbol PCF8563
Connections:
- net at IC1.27 ((PCINT12/SDA/ADC4)PC4): now also U?.5 (SDA)
- net at IC1.28 ((PCINT13/SCL/ADC5)PC5): now also U?.6 (SCL)
Changed lines of the file:
@@
 Wire Wire Line
 	4000 5500 800  5500
+$Comp
+L PCF8563 U?
+U 1 1 58F25C8C
+P 6350 1700
+F 0 "U?" H 6050 2050 50  0000 L CNN
+F 1 "PCF8563" H 6450 2050 50  0000 L CNN
+F 2 "" H 6350 1700 50  0001 C CNN
+F 3 "" H 6350 1700 50  0001 C CNN
+	1    6350 1700
+	1    0    0    -1
+$EndComp
+Wire Wire Line
+	2750 2450 2900 2450
+Wire Wire Line
+	2900 2450 2900 900
+Wire Wire Line
+	2900 900  7100 900
+Wire Wire Line
+	7100 900  7100 1600
+Wire Wire Line
+	7100 1600 6750 1600
+Wire Wire Line
+	2750 2550 3000 2550
+Wire Wire Line
+	3000 2550 3000 1000
+Wire Wire Line
+	3000 1000 7000 1000
+Wire Wire Line
+	7000 1000 7000 1500
+Wire Wire Line
+	7000 1500 6750 1500
 $EndSCHEMATC

Commit message: update kicad
Parts:
- added Y2: 32768kHz, symbol Crystal
- gave numbers to parts that had none: 1
Connections:
- net at U4.1 (OSCI): now also Y2.1
- net at U4.2 (OSCO): now also Y2.2
Changed lines of the file:
@@
 $EndComp
 $Comp
-L +5V #PWR01
+L +5V #PWR1
 U 1 1 5683D91E
 P 600 700
-F 0 "#PWR01" H 600 550 50  0001 C CNN
+F 0 "#PWR1" H 600 550 50  0001 C CNN
 F 1 "+5V" H 600 840 50  0000 C CNN
 F 2 "" H 600 700 50  0000 C CNN
@@
 $EndComp
 $Comp
-L Earth #PWR02
+L Earth #PWR2
 U 1 1 58ED2D1B
 P 600 3850
-F 0 "#PWR02" H 600 3600 50  0001 C CNN
+F 0 "#PWR2" H 600 3600 50  0001 C CNN
 F 1 "Earth" H 600 3700 50  0001 C CNN
 F 2 "" H 600 3850 50  0001 C CNN
@@
 $EndComp
 $Comp
-L Earth #PWR03
+L Earth #PWR5
 U 1 1 58ED2D67
 P 4550 3000
-F 0 "#PWR03" H 4550 2750 50  0001 C CNN
+F 0 "#PWR5" H 4550 2750 50  0001 C CNN
 F 1 "Earth" H 4550 2850 50  0001 C CNN
 F 2 "" H 4550 3000 50  0001 C CNN
@@
 $EndComp
 $Comp
-L Earth #PWR04
+L Earth #PWR6
 U 1 1 58EF5DC6
 P 4550 8800
-F 0 "#PWR04" H 4550 8550 50  0001 C CNN
+F 0 "#PWR6" H 4550 8550 50  0001 C CNN
 F 1 "Earth" H 4550 8650 50  0001 C CNN
 F 2 "" H 4550 8800 50  0001 C CNN
@@
 $EndComp
 $Comp
-L Earth #PWR?
+L Earth #PWR4
 U 1 1 58EF99D1
 P 700 9550
-F 0 "#PWR?" H 700 9300 50  0001 C CNN
+F 0 "#PWR4" H 700 9300 50  0001 C CNN
 F 1 "Earth" H 700 9400 50  0001 C CNN
 F 2 "" H 700 9550 50  0001 C CNN
@@
 $EndComp
 $Comp
-L +5V #PWR?
+L +5V #PWR3
 U 1 1 58EF9ECF
 P 600 5300
-F 0 "#PWR?" H 600 5150 50  0001 C CNN
+F 0 "#PWR3" H 600 5150 50  0001 C CNN
 F 1 "+5V" H 600 5440 50  0000 C CNN
 F 2 "" H 600 5300 50  0001 C CNN
@@
 	4000 5500 800  5500
 $Comp
-L PCF8563 U?
+L PCF8563 U4
 U 1 1 58F25C8C
 P 6350 1700
-F 0 "U?" H 6050 2050 50  0000 L CNN
+F 0 "U4" H 6050 2050 50  0000 L CNN
 F 1 "PCF8563" H 6450 2050 50  0000 L CNN
 F 2 "" H 6350 1700 50  0001 C CNN
@@
 Wire Wire Line
 	7000 1500 6750 1500
+$Comp
+L Crystal Y2
+U 1 1 58F49E8C
+P 5850 1700
+F 0 "Y2" H 5850 1850 50  0000 C CNN
+F 1 "32768kHz" H 5850 1550 50  0000 C CNN
+F 2 "" H 5850 1700 50  0001 C CNN
+F 3 "" H 5850 1700 50  0001 C CNN
+	1    5850 1700
+	0    1    1    0
+$EndComp
+Wire Wire Line
+	5850 1550 5850 1500
+Wire Wire Line
+	5850 1500 5950 1500
+Wire Wire Line
+	5850 1850 5850 1900
+Wire Wire Line
+	5850 1900 5950 1900
 $EndSCHEMATC

Commit message: update kicad
Parts:
- added D25, D26: 1N4148, symbol D
Connections:
- net +5V: now also D25.2 (A)
- net Earth: now also U4.4 (VSS)
- net at U4.8 (VDD): now also D25.1 (K), D26.1 (K)
- new net +3V3: D26.2 (A)
Changed lines of the file:
@@
 Wire Wire Line
 	5850 1900 5950 1900
+$Comp
+L Earth #PWR8
+U 1 1 5902180B
+P 6350 2350
+F 0 "#PWR8" H 6350 2100 50  0001 C CNN
+F 1 "Earth" H 6350 2200 50  0001 C CNN
+F 2 "" H 6350 2350 50  0001 C CNN
+F 3 "" H 6350 2350 50  0001 C CNN
+	1    6350 2350
+	1    0    0    -1
+$EndComp
+$Comp
+L +5V #PWR7
+U 1 1 5902186D
+P 5950 1200
+F 0 "#PWR7" H 5950 1050 50  0001 C CNN
+F 1 "+5V" H 5950 1340 50  0000 C CNN
+F 2 "" H 5950 1200 50  0001 C CNN
+F 3 "" H 5950 1200 50  0001 C CNN
+	1    5950 1200
+	1    0    0    -1
+$EndComp
+$Comp
+L +3.3V #PWR9
+U 1 1 59021B22
+P 6750 1200
+F 0 "#PWR9" H 6750 1050 50  0001 C CNN
+F 1 "+3.3V" H 6750 1340 50  0000 C CNN
+F 2 "" H 6750 1200 50  0001 C CNN
+F 3 "" H 6750 1200 50  0001 C CNN
+	1    6750 1200
+	1    0    0    -1
+$EndComp
+$Comp
+L D D26
+U 1 1 59021B84
+P 6550 1200
+F 0 "D26" H 6550 1300 50  0000 C CNN
+F 1 "1N4148" H 6550 1100 50  0000 C CNN
+F 2 "" H 6550 1200 50  0001 C CNN
+F 3 "" H 6550 1200 50  0001 C CNN
+	1    6550 1200
+	1    0    0    -1
+$EndComp
+$Comp
+L D D25
+U 1 1 59021C21
+P 6150 1200
+F 0 "D25" H 6150 1300 50  0000 C CNN
+F 1 "1N4148" H 6150 1100 50  0000 C CNN
+F 2 "" H 6150 1200 50  0001 C CNN
+F 3 "" H 6150 1200 50  0001 C CNN
+	1    6150 1200
+	-1   0    0    1
+$EndComp
+Wire Wire Line
+	5950 1200 6000 1200
+Wire Wire Line
+	6300 1200 6400 1200
+Wire Wire Line
+	6350 1300 6350 1200
+Connection ~ 6350 1200
+Wire Wire Line
+	6700 1200 6750 1200
+Wire Wire Line
+	6350 2350 6350 2100
 $EndSCHEMATC

Commit message: update kicad
Parts:
- added R? (x2): R, symbol R
Connections:
- net at IC1.27 ((PCINT12/SDA/ADC4)PC4), U4.5 (SDA): now also R?.2
- net at IC1.28 ((PCINT13/SCL/ADC5)PC5), U4.6 (SCL): now also R?.2
- net at D25.1 (K), D26.1 (K), U4.8 (VDD): now also R?.1, R?.1
