File: kicad/binaryclock.sch (KiCad schematic (older format))
At the start: 43 parts, among them IC1 ATMEGA328P-PU, SW1 Reset, U1 74HC595, U2 74HC595, U3 74HC595, U4 PCF8563, Y1 16MHz, Y2 32768kHz

Commit message: update kicad
Parts:
- R? (x2): value R -> 10KΩ
Changed lines of the file:
@@
 P 5850 600
 F 0 "R?" V 5930 600 50  0000 C CNN
-F 1 "R" V 5850 600 50  0000 C CNN
+F 1 "10KΩ" V 5850 600 50  0000 C CNN
 F 2 "" V 5780 600 50  0001 C CNN
 F 3 "" H 5850 600 50  0001 C CNN
@@
 P 5850 800
 F 0 "R?" V 5930 800 50  0000 C CNN
-F 1 "R" V 5850 800 50  0000 C CNN
+F 1 "10KΩ" V 5850 800 50  0000 C CNN
 F 2 "" V 5780 800 50  0001 C CNN
 F 3 "" H 5850 800 50  0001 C CNN
